Commit message: fix: Fix robot orientation and create new custom plugin to integrate the robot kinematic producing a faster simulation.

File: 0_mindstorm_simulator/1_lego_robot/urdf/my_robot.xacro (robot description, xacro)
@@ -14,27 +14,12 @@
   <link name="robot_footprint"></link>
   <joint name="robot_footprint_joint" type="fixed">
-    <origin xyz="0 0 0" rpy="0 0 -3.14" />
+    <origin xyz="0 0 0" rpy="0 0 0" />
     <parent link="robot_footprint"/>
     <child link="chassis" />
   </joint>
-  <joint name="robot_top_triangle_joint" type="fixed">
-    <origin xyz="0 0 0" rpy="0 0 0" />
-    <parent link="chassis"/>
-    <child link="top_triangle" />
-  </joint>
-  <joint name="robot_top_layer_joint" type="fixed">
-    <origin xyz="0 0 0" rpy="0 0 0" />
-    <parent link="chassis"/>
-    <child link="top_layer" />
-  </joint>
-  <joint name="robot_NXT20_joint" type="fixed">
-    <origin xyz="0 0 0" rpy="0 0 0" />
-    <parent link="chassis"/>
-    <child link="NXT20" />
-  </joint>
   <link name='chassis'>
     <inertial>
-      <mass value="1.5"/>
-      <origin xyz="${footprint_length/2 - axel_dx} 0 ${wheel_radius}" rpy=" 0 0 0"/>
+      <mass value="5.0"/>
+      <origin xyz="${-footprint_length/2 + axel_dx} 0 0" rpy=" 0 0 0"/>
       <inertia
           ixx="0.001" ixy="0" ixz="0"
@@ -44,5 +29,5 @@
     </inertial>
     <collision name='chassis_collision'>
-      <origin xyz="${footprint_length/2 - axel_dx} 0 ${wheel_radius}" rpy=" 0 0 0"/>
+      <origin xyz="${-footprint_length/2 + axel_dx} 0 ${wheel_radius}" rpy=" 0 0 0"/>
       <geometry>
         <box size="${footprint_length} ${footprint_width} ${footprint_height}"/>
@@ -50,5 +35,5 @@
     </collision>
     <visual name='chassis_visual'>
-      <origin xyz="${footprint_length/2 - axel_dx} 0 ${wheel_radius}" rpy=" 0 0 0"/>
+      <origin xyz="${-footprint_length/2 + axel_dx} 0 ${wheel_radius}" rpy=" 0 0 0"/>
       <geometry>
         <box size="${footprint_length} ${footprint_width} ${footprint_height}"/>
@@ -56,5 +41,5 @@
     </visual>
      <collision name='back_caster_collision'>
-      <origin xyz="${footprint_length - axel_dx - wheel_radius} 0 ${wheel_radius}" rpy=" 0 0 0"/>
+      <origin xyz="${-footprint_length + axel_dx + wheel_radius} 0 ${wheel_radius}" rpy=" 0 0 0"/>
       <geometry>
         <sphere radius="${wheel_radius}"/>
@@ -72,25 +57,18 @@
     </collision>
     <visual name='back_caster_visual'>
-      <origin xyz="${footprint_length - axel_dx - wheel_radius} 0 ${wheel_radius}" rpy=" 0 0 0"/>
+      <origin xyz="${-footprint_length + axel_dx + wheel_radius} 0 ${wheel_radius}" rpy=" 0 0 0"/>
       <geometry>
         <sphere radius="${wheel_radius}"/>
       </geometry>
     </visual>
-    <!--collision name='nxt_collision'>
-      <origin xyz="${triangle_h/6 + 0.005} 0 ${triangle_z - 0.005}" rpy=" 0 0 0"/>
-      <geometry>
-        <box size="${triangle_h} ${triangle_b} 0.01"/>
-      </geometry>
-    </collision>
-    <visual name='nxt_visual'>
-      <origin xyz="${triangle_h/6 + 0.005} 0 ${triangle_z - 0.005}" rpy=" 0 0 0"/>
-      <geometry>
-        <box size="${triangle_h} ${triangle_b} 0.01"/>
-      </geometry>
-    </visual-->
-  </link>
+  </link>
+  <joint name="robot_NXT20_joint" type="fixed">
+    <origin xyz="0 0 0" rpy="0 0 0" />
+    <parent link="chassis"/>
+    <child link="NXT20" />
+  </joint>
   <link name="NXT20">
     <visual name='NXT20_visual'>
-      <origin xyz="0.05 0 ${triangle_z/2}" rpy="-0.7853 0 1.5707"/>
+      <origin xyz="-0.05 0 ${triangle_z/2}" rpy="-0.7853 0 -1.5707"/>
       <geometry>
         <mesh filename="package://lego_robot/media/models/Lego_MindstormsNXT20.stl"  scale="0.001 0.001 0.001"/>
@@ -99,7 +77,12 @@
     </visual>
   </link>
+  <joint name="robot_top_layer_joint" type="fixed">
+    <origin xyz="0 0 0" rpy="0 0 0" />
+    <parent link="chassis"/>
+    <child link="top_layer" />
+  </joint>
   <link name="top_layer">
       <collision name='top_layer_collision'>
-      <origin xyz="${triangle_h/6 + 0.005} 0 ${triangle_z - 0.005}" rpy=" 0 0 0"/>
+      <origin xyz="${-triangle_h/6} 0 ${triangle_z - 0.005}" rpy=" 0 0 0"/>
       <geometry>
         <box size="${triangle_h} ${triangle_b} 0.005"/>
@@ -107,5 +90,5 @@
     </collision>
     <visual name='top_layer_visual'>
-     <origin xyz="${triangle_h/6 + 0.005} 0 ${triangle_z - 0.005}" rpy=" 0 0 0"/>
+     <origin xyz="${-triangle_h/6} 0 ${triangle_z - 0.005}" rpy=" 0 0 0"/>
       <geometry>
         <box size="${triangle_h} ${triangle_b} 0.005"/>
@@ -113,7 +96,12 @@
     </visual>
   </link>
+  <joint name="robot_top_triangle_joint" type="fixed">
+    <origin xyz="0 0 0" rpy="0 0 0" />
+    <parent link="chassis"/>
+    <child link="top_triangle" />
+  </joint>
   <link name="top_triangle">
       <collision name='top_layer_collision'>
-      <origin xyz="${triangle_h/6 + 0.005} 0 ${triangle_z - 0.0025}" rpy=" 0 0 0"/>
+      <origin xyz="${-triangle_h/6 + triangle_h/2 } 0 ${triangle_z - 0.0025}" rpy=" 0 0 3.1415"/>
       <geometry>
         <box size="${triangle_h} ${triangle_b} 0.005"/>
@@ -121,8 +109,7 @@
     </collision>
     <visual name='top_triangle_visual'>
-      <origin xyz="${-0.16/3 + 0.005} -0.04 ${triangle_z - 0.01}" rpy=" 0 0 0"/>
+      <origin xyz="${-triangle_h/6 + triangle_h/2} 0.04 ${triangle_z - 0.01}" rpy=" 0 0 3.1415"/>
       <geometry>
         <mesh filename="package://lego_robot/media/models/triangle.STL"  scale="0.001 0.001 0.001"/>
-        <!--box size="${triangle_h} ${triangle_b} 0.005"/-->
       </geometry>
     </visual>
@@ -142,5 +129,5 @@
     </visual>
     <inertial>
-      <mass value="0.1"/>
+      <mass value="1"/>
       <origin xyz="0.0 0 0" rpy="0 1.5707 1.5707"/>
       <inertia
@@ -165,5 +152,5 @@
     </visual>
     <inertial>
-      <mass value="0.1"/>
+      <mass value="1"/>
       <origin xyz="0.0 0 0" rpy="0 1.5707 1.5707"/>
       <inertia
@@ -175,17 +162,17 @@
   </link>
   <joint type="continuous" name="left_wheel_hinge">
-    <origin xyz="0 ${footprint_width/2} ${wheel_radius}" rpy="0 0 0"/>
+    <origin xyz="0 ${footprint_width/2 + 0.001} ${wheel_radius}" rpy="0 0 0"/>
     <child link="left_wheel"/>
     <parent link="chassis"/>
-    <axis xyz="0 -1 0" rpy="0 0 0"/>
-    <limit effort="5" velocity="100"/>
+    <axis xyz="0 1 0" rpy="0 0 0"/>
+    <limit effort="1000" velocity="1000"/>
     <dynamics damping="0.0" friction="0.0"/>
   </joint>
   <joint type="continuous" name="right_wheel_hinge">
-    <origin xyz="0 ${-footprint_width/2} ${wheel_radius}" rpy="0 0 0"/>
+    <origin xyz="0 ${-footprint_width/2 - 0.001} ${wheel_radius}" rpy="0 0 0"/>
     <child link="right_wheel"/>
     <parent link="chassis"/>
-    <axis xyz="0 -1 0" rpy="0 0 0"/>
-    <limit effort="5" velocity="100"/>
+    <axis xyz="0 1 0" rpy="0 0 0"/>
+    <limit effort="1000" velocity="1000"/>
     <dynamics damping="0.0" friction="0.0"/>
   </joint>

Commit message: fix: fixed frame name in visualization and world

File: 0_mindstorm_simulator/1_lego_robot/urdf/my_robot.xacro (robot description, xacro)
@@ -121,4 +121,14 @@
         <cylinder radius="${wheel_radius}" length="${wheel_width}"/>
       </geometry>
+      <surface>
+        <friction>
+          <ode>
+            <mu>0</mu>
+            <mu2>0</mu2>
+            <slip1>1.0</slip1>
+            <slip2>1.0</slip2>
+          </ode>
+        </friction>
+      </surface>
     </collision>
     <visual name='left_wheel_visual'>
@@ -145,4 +155,14 @@
       </geometry>
     </collision>
+    <surface>
+      <friction>
+        <ode>
+          <mu>0</mu>
+          <mu2>0</mu2>
+          <slip1>1.0</slip1>
+          <slip2>1.0</slip2>
+        </ode>
+      </friction>
+    </surface>
     <visual name='right_wheel_visual'>
       <origin xyz="0 ${-wheel_width/2} 0" rpy="0 1.5707 1.5707"/>
@@ -161,19 +181,19 @@
     </inertial>
   </link>
-  <joint type="continuous" name="left_wheel_hinge">
+  <joint type="fixed" name="left_wheel_hinge">
     <origin xyz="0 ${footprint_width/2 + 0.001} ${wheel_radius}" rpy="0 0 0"/>
     <child link="left_wheel"/>
     <parent link="chassis"/>
-    <axis xyz="0 1 0" rpy="0 0 0"/>
+    <!--axis xyz="0 1 0" rpy="0 0 0"/>
     <limit effort="1000" velocity="1000"/>
-    <dynamics damping="0.0" friction="0.0"/>
-  </joint>
-  <joint type="continuous" name="right_wheel_hinge">
+    <dynamics damping="0.0" friction="0.0"/-->
+  </joint>
+  <joint type="fixed" name="right_wheel_hinge">
     <origin xyz="0 ${-footprint_width/2 - 0.001} ${wheel_radius}" rpy="0 0 0"/>
     <child link="right_wheel"/>
     <parent link="chassis"/>
-    <axis xyz="0 1 0" rpy="0 0 0"/>
+    <!--axis xyz="0 1 0" rpy="0 0 0"/>
     <limit effort="1000" velocity="1000"/>
-    <dynamics damping="0.0" friction="0.0"/>
+    <dynamics damping="0.0" friction="0.0"/-->
   </joint>
 <gazebo reference="left_wheel">
